Commit message: added GPS, IMU links to URDF

File: description/robot_core.xacro (robot description, xacro)
@@ -149,3 +149,15 @@
         <mu2 value="0.001"/>
     </gazebo>
+    <joint name="imu_joint" type="fixed">
+        <parent link="base_link"/>
+        <child link="imu_link"/>
+        <origin xyz="-40 83 530" rpy="0 0 0"/>
+    </joint>
+    <link name="imu_link"/>
+    <joint name="gps_joint" type="fixed">
+        <parent link="base_link"/>
+        <child link="gps_link"/>
+        <origin xyz="40 0 320" rpy="0 0 0"/>
+    </joint>
+    <link name="gps_link"/>
 </robot>

Commit message: fixed units to meters

File: description/robot_core.xacro (robot description, xacro)
@@ -152,5 +152,5 @@
         <parent link="base_link"/>
         <child link="imu_link"/>
-        <origin xyz="-40 83 530" rpy="0 0 0"/>
+        <origin xyz="-0.040 0.083 0.530" rpy="0 0 0"/>
     </joint>
     <link name="imu_link"/>
@@ -158,5 +158,5 @@
         <parent link="base_link"/>
         <child link="gps_link"/>
-        <origin xyz="40 0 320" rpy="0 0 0"/>
+        <origin xyz="0.040 0 0.320" rpy="0 0 0"/>
     </joint>
     <link name="gps_link"/>

Commit message: corrected imu, gps position in URDF

File: description/robot_core.xacro (robot description, xacro)
@@ -152,5 +152,5 @@
         <parent link="base_link"/>
         <child link="imu_link"/>
-        <origin xyz="-0.040 0.083 0.530" rpy="0 0 0"/>
+        <origin xyz="0.040 -0.083 0.530" rpy="0 0 0"/>
     </joint>
     <link name="imu_link"/>
@@ -158,5 +158,5 @@
         <parent link="base_link"/>
         <child link="gps_link"/>
-        <origin xyz="0.040 0 0.320" rpy="0 0 0"/>
+        <origin xyz="-0.040 0 0.320" rpy="0 0 0"/>
     </joint>
     <link name="gps_link"/>

Commit message: disabled odom tf for gps nav + fixed wheel size

File: description/robot_core.xacro (robot description, xacro)
@@ -37,6 +37,6 @@
     <!-- BASE_FOOTPRINT LINK -->
     <joint name="base_footprint_joint" type="fixed">
-        <parent link="base_link"/>
-        <child link="base_footprint"/>
+        <parent link="base_footprint"/>
+        <child link="base_link"/>
         <origin xyz="0 0 0" rpy="0 0 0"/>
     </joint>
