Commit message: fixed ultrasonic position

File: description/dual_ultrasonic.xacro (robot description, xacro)
@@ -4,5 +4,5 @@
         <parent link="base_link"/>
         <child link="range_box_link"/>
-        <origin xyz="0.040 0 0.040" rpy="0 0 0"/>
+        <origin xyz="0.115 0 0.040" rpy="0 0 0"/>
     </joint>
     <link name="range_box_link">
