Commit message: corrected typo (height)

File: description/mower2_core.xacro (robot description, xacro)
@@ -27,10 +27,10 @@
     <xacro:property name="main_box_offset_z" value="${chassis_height}"/>
     <xacro:property name="main_box_length" value="0.292"/>
-    <xacro:property name="main_box_heigth" value="0.099"/>
+    <xacro:property name="main_box_height" value="0.099"/>
     <xacro:property name="main_box_width" value="0.20"/>
     <xacro:property name="gps_box_offset_x" value="0.190"/>
-    <xacro:property name="gps_box_offset_z" value="${chassis_height} + ${main_box_heigth}"/>
+    <xacro:property name="gps_box_offset_z" value="${chassis_height} + ${main_box_height}"/>
     <xacro:property name="gps_box_length" value="0.140"/>
-    <xacro:property name="gps_box_heigth" value="0.193"/>
+    <xacro:property name="gps_box_height" value="0.193"/>
     <xacro:property name="gps_box_width" value="0.196"/>
     <xacro:property name="imu_cylinder_offset_x" value="${chassis_length} - 0.022"/>

Commit message: corrected urdf pos params

File: description/mower2_core.xacro (robot description, xacro)
@@ -30,10 +30,10 @@
     <xacro:property name="main_box_width" value="0.20"/>
     <xacro:property name="gps_box_offset_x" value="0.190"/>
-    <xacro:property name="gps_box_offset_z" value="${chassis_height} + ${main_box_height}"/>
+    <xacro:property name="gps_box_offset_z" value="${chassis_height + main_box_height}"/>
     <xacro:property name="gps_box_length" value="0.140"/>
     <xacro:property name="gps_box_height" value="0.193"/>
     <xacro:property name="gps_box_width" value="0.196"/>
-    <xacro:property name="imu_cylinder_offset_x" value="${chassis_length} - 0.022"/>
-    <xacro:property name="imu_cylinder_offset_y" value="${chassis_widht}/2 - 0.017"/>
+    <xacro:property name="imu_cylinder_offset_x" value="${chassis_length - 0.022}"/>
+    <xacro:property name="imu_cylinder_offset_y" value="${chassis_width/2 - 0.017}"/>
     <xacro:property name="imu_cylinder_offset_z" value="${chassis_height}"/>
     <xacro:property name="imu_cylinder_length" value="0.506"/>

Commit message: URDF - caster wheel and imu pole fix

File: description/mower2_core.xacro (robot description, xacro)
@@ -19,5 +19,5 @@
     <xacro:property name="wheel_offset_z" value="0.013"/>
     <!-- <xacro:property name="caster_wheel_radius" value="0.01"/> -->
-    <xacro:property name="caster_wheel_radius" value="0.051"/>
+    <xacro:property name="caster_wheel_radius" value="${0.051 / 2}"/>
     <xacro:property name="caster_wheel_mass" value="0.01"/>
     <!-- <xacro:property name="caster_wheel_offset_x" value="0.075"/> -->
@@ -35,8 +35,8 @@
     <xacro:property name="gps_box_width" value="0.196"/>
     <xacro:property name="imu_cylinder_offset_x" value="${chassis_length - 0.022}"/>
-    <xacro:property name="imu_cylinder_offset_y" value="${chassis_width/2 - 0.017}"/>
+    <xacro:property name="imu_cylinder_offset_y" value="${-chassis_width/2 + 0.017}"/>
     <xacro:property name="imu_cylinder_offset_z" value="${chassis_height}"/>
     <xacro:property name="imu_cylinder_length" value="0.506"/>
-    <xacro:property name="imu_cylinder_radius" value="0.120"/>
+    <xacro:property name="imu_cylinder_radius" value="0.012"/>
     <material name="white">
         <color rgba="1 1 1 1" />

Commit message: URDF IMU pole position

File: description/mower2_core.xacro (robot description, xacro)
@@ -34,9 +34,9 @@
     <xacro:property name="gps_box_height" value="0.193"/>
     <xacro:property name="gps_box_width" value="0.196"/>
+    <xacro:property name="imu_cylinder_length" value="0.506"/>
+    <xacro:property name="imu_cylinder_radius" value="0.012"/>
     <xacro:property name="imu_cylinder_offset_x" value="${chassis_length - 0.022}"/>
     <xacro:property name="imu_cylinder_offset_y" value="${-chassis_width/2 + 0.017}"/>
-    <xacro:property name="imu_cylinder_offset_z" value="${chassis_height}"/>
-    <xacro:property name="imu_cylinder_length" value="0.506"/>
-    <xacro:property name="imu_cylinder_radius" value="0.012"/>
+    <xacro:property name="imu_cylinder_offset_z" value="${chassis_height + imu_cylinder_length/2}"/>
     <material name="white">
         <color rgba="1 1 1 1" />

Commit message: added visual GPS,IMU links

File: description/mower2_core.xacro (robot description, xacro)
@@ -204,5 +204,13 @@
         <origin xyz="0.040 -0.083 0.530" rpy="0 0 0"/>
     </joint>
-    <link name="imu_link"/>
+    <link name="imu_link">
+        <visual>
+            <origin xyz="0 0 0"/>
+            <geometry>
+                <box size="0.02 0.02 0.005"/>
+            </geometry>
+            <material name="black"/>
+        </visual>
+    </link>
     <joint name="imu_cyl_joint" type="fixed">
         <parent link="chassis"/>
@@ -227,5 +235,13 @@
         <origin xyz="-0.040 0 0.320" rpy="0 0 0"/>
     </joint>
-    <link name="gps_link"/>
+    <link name="gps_link">
+        <visual>
+            <origin xyz="0 0 0.005"/>
+            <geometry>
+                <box size="0.04 0.04 0.01"/>
+            </geometry>
+            <material name="black"/>
+        </visual>
+    </link>
     <joint name="gps_box_joint" type="fixed">
         <parent link="chassis"/>

Commit message: URDF - corrected chassis position

File: description/mower2_core.xacro (robot description, xacro)
@@ -69,5 +69,5 @@
         <parent link="base_link"/>
         <child link="chassis"/>
-        <origin xyz="${-wheel_offset_x} 0 ${-wheel_offset_z}"/>
+        <origin xyz="${-wheel_offset_x} 0 ${wheel_offset_z}"/>
     </joint>
     <link name="chassis">

Commit message: URDF - corrected caster wheel pos

File: description/mower2_core.xacro (robot description, xacro)
@@ -23,5 +23,5 @@
     <!-- <xacro:property name="caster_wheel_offset_x" value="0.075"/> -->
     <xacro:property name="caster_wheel_offset_x" value="0.032"/>
-    <xacro:property name="caster_wheel_offset_z" value="${wheel_offset_z - wheel_radius + caster_wheel_radius}"/>
+    <xacro:property name="caster_wheel_offset_z" value="${-wheel_offset_z - wheel_radius + caster_wheel_radius}"/>
     <xacro:property name="main_box_offset_x" value="0.028"/>
     <xacro:property name="main_box_offset_z" value="${chassis_height}"/>
